Commit message: gripper needed

File: mm_description/urdf/mm.urdf.xacro (robot description, xacro)
@@ -1,54 +1,16 @@
 <?xml version="1.0"?>
-<robot name="mm_robot" xmlns:xacro="http://ros.org/wiki/xacro">
-    <!-- Included URDF/XACRO Files -->
-    <xacro:include filename="$(find mm_description)/urdf/components/wheels.urdf.xacro" />
-    <xacro:include filename="$(find mm_description)/urdf/components/chassis.urdf.xacro" />
-    <xacro:include filename="$(find mm_description)/urdf/sensors/kinect.urdf.xacro" />
-    <!-- Add UR5 -->
-    <xacro:property name="M_PI" value="3.14159"/>
-    <!-- Wheel Mounting Positions -->
-    <xacro:property name="track" value="0.48122440" />
-    <xacro:property name="wheel_vertical_offset" value="0.08255015" />
-    <!-- Wheel Properties -->
-    <xacro:property name="wheel_length" value="0.09224900" />
-    <xacro:property name="wheel_radius" value="0.2405681" />
-    <xacro:macro name="mm_robot">
-        <!-- Base link is the center of the robot's chassis between the motors projected on the ground -->
-        <link name="base_link"/>
-        <!--Chassis -->
-        <xacro:chassis chassis_prefix="base" parent="base_link">
-            <origin xyz="0 0 ${-wheel_vertical_offset + wheel_radius}" rpy="0 0 0" />
-        </xacro:chassis>
-        <link name="inertial_collision_link">
-			<inertial>
-				<mass value="29.756375" />
-				<origin xyz="0.001751 0.000008 0.018544" />
-				<inertia ixx="0.696269"  ixy="0.016133" ixz="0.003232"
-                         iyx="0.016133"  iyy="0.299110" iyz="-0.000004"
-                         izx="-0.077476" izy="-0.000004" izz="0.864394" />
-			</inertial>
-            <collision>
-				<geometry>
-					<mesh filename="package://mm_description/meshes/collision/chassis.stl" />
-				</geometry>
-			</collision>
-		</link>
-		<joint name="inertial_collision_joint" type="fixed" >
-		    <parent link="base_chassis_link" />
-		    <child link="inertial_collision_link" />
-		</joint>
-        <!-- Wheel macros -->
-        <xacro:wheel wheel_prefix="left" parent="base_chassis_link" visual_rotation="0.0">
-            <origin xyz="0 ${track/2} ${wheel_vertical_offset}" rpy="0 0 0" />
-        </xacro:wheel>
-        <xacro:wheel wheel_prefix="left" parent="base_chassis_link" visual_rotation="0.0">
-            <origin xyz="0 ${track/2} ${wheel_vertical_offset}" rpy="0 0 0" />
-        </xacro:wheel>
-        <xacro:wheel wheel_prefix="left" parent="base_chassis_link" visual_rotation="0.0">
-            <origin xyz="0 ${track/2} ${wheel_vertical_offset}" rpy="0 0 0" />
-        </xacro:wheel>
-        <xacro:wheel wheel_prefix="left" parent="base_chassis_link" visual_rotation="0.0">
-            <origin xyz="0 ${track/2} ${wheel_vertical_offset}" rpy="0 0 0" />
-        </xacro:wheel>
-    </xacro:macro>
+<robot name="inspector_bot" xmlns:xacro="http://ros.org/wiki/xacro">
+  <xacro:arg name="robot_namespace" default="/" />
+  <!-- Included URDF/XACRO Files -->
+  <xacro:include filename="$(find mm_description)/urdf/components/inspector_bot.urdf.xacro" />
+  <xacro:include filename="$(find ur_description)/urdf/ur5.urdf.xacro" />
+  <xacro:property name="ur5_z_location" value="${base_center_height + base_z_size/2}" />
+  <xacro:property name="ur5_x_location" value="0.2" />
+  <xacro:bare_base/>
+  <xacro:ur5_robot prefix="" joint_limited="false"/>
+  <joint name="ur_fixed_joint" type="fixed">
+    <parent link="bare_base_link" />
+    <child link = "base_link" />
+    <origin xyz="${ur5_x_location} 0.0 ${ur5_z_location}" rpy="0.0 0.0 ${M_PI/2}  " />
+  </joint>
 </robot>

Commit message: gripper added

File: mm_description/urdf/mm.urdf.xacro (robot description, xacro)
@@ -5,8 +5,11 @@
   <xacro:include filename="$(find mm_description)/urdf/components/inspector_bot.urdf.xacro" />
   <xacro:include filename="$(find ur_description)/urdf/ur5.urdf.xacro" />
+  <xacro:include filename="$(find robotiq_arg2f_model_visualization)/urdf/robotiq_arg2f_140_model_macro.xacro" />
   <xacro:property name="ur5_z_location" value="${base_center_height + base_z_size/2}" />
   <xacro:property name="ur5_x_location" value="0.2" />
+  <xacro:property name="gripper_z_location_ee" value="0.08" />
   <xacro:bare_base/>
   <xacro:ur5_robot prefix="" joint_limited="false"/>
+  <xacro:robotiq_arg2f_140 prefix=""/>
   <joint name="ur_fixed_joint" type="fixed">
     <parent link="bare_base_link" />
@@ -14,3 +17,8 @@
     <origin xyz="${ur5_x_location} 0.0 ${ur5_z_location}" rpy="0.0 0.0 ${M_PI/2}  " />
   </joint>
+  <joint name="ur_gripper_fixed_joint" type="fixed">
+    <parent link="wrist_3_link" />
+    <child link = "robotiq_arg2f_base_link" />
+    <origin xyz="0.0 ${gripper_z_location_ee} 0.0" rpy="${-M_PI/2} 0.0 0.0  " />
+  </joint>
 </robot>

Commit message: kinect added

File: mm_description/urdf/mm.urdf.xacro (robot description, xacro)
@@ -6,7 +6,11 @@
   <xacro:include filename="$(find ur_description)/urdf/ur5.urdf.xacro" />
   <xacro:include filename="$(find robotiq_arg2f_model_visualization)/urdf/robotiq_arg2f_140_model_macro.xacro" />
+  <xacro:include filename="$(find mm_description)/urdf/accessories/kinect_camera.urdf.xacro"/>
   <xacro:property name="ur5_z_location" value="${base_center_height + base_z_size/2}" />
   <xacro:property name="ur5_x_location" value="0.2" />
   <xacro:property name="gripper_z_location_ee" value="0.08" />
+  <xacro:arg name="kinect_enabled" default="false" />
+  <xacro:arg name="kinect_xyz" default="$(optenv MM_KINECT_XYZ ${base_x_size/2 + 0.03}  ${-base_y_size/2 + 0.12}  ${ur5_z_location - 0.03} )" />
+  <xacro:arg name="kinect_rpy" default="$(optenv MM_KINECT_RPY 0 0.0 0.0)" />
   <xacro:bare_base/>
   <xacro:ur5_robot prefix="" joint_limited="false"/>
@@ -22,3 +26,11 @@
     <origin xyz="0.0 ${gripper_z_location_ee} 0.0" rpy="${-M_PI/2} 0.0 0.0  " />
   </joint>
+  <xacro:if value="$(arg kinect_enabled)">
+    <joint name="kinect_frame_joint" type="fixed">
+      <origin xyz="$(arg kinect_xyz)" rpy="$(arg kinect_rpy)" />
+      <parent link="bare_base_link"/>
+      <child link="camera_link"/>
+    </joint>
+    <xacro:kinect_camera prefix="camera" robot_namespace="$(arg robot_namespace)"/>
+  </xacro:if>
 </robot>

Commit message: disconnected arg2f from the system

File: mm_description/urdf/mm.urdf.xacro (robot description, xacro)
@@ -5,5 +5,5 @@
   <xacro:include filename="$(find mm_description)/urdf/components/inspector_bot.urdf.xacro" />
   <xacro:include filename="$(find ur_description)/urdf/ur5.urdf.xacro" />
-  <xacro:include filename="$(find robotiq_arg2f_model_visualization)/urdf/robotiq_arg2f_140_model_macro.xacro" />
+  <!-- <xacro:include filename="$(find robotiq_arg2f_model_visualization)/urdf/robotiq_arg2f_140_model_macro.xacro" /> -->
   <xacro:include filename="$(find mm_description)/urdf/accessories/kinect_camera.urdf.xacro"/>
   <xacro:property name="ur5_z_location" value="${base_center_height + base_z_size/2}" />
@@ -11,9 +11,9 @@
   <xacro:property name="gripper_z_location_ee" value="0.08" />
   <xacro:arg name="kinect_enabled" default="false" />
-  <xacro:arg name="kinect_xyz" default="$(optenv MM_KINECT_XYZ ${base_x_size/2 + 0.03}  ${-base_y_size/2 + 0.12}  ${ur5_z_location - 0.03} )" />
+  <xacro:arg name="kinect_xyz" default="$(optenv MM_KINECT_XYZ ${base_x_size/2 + 0.03 + 0.025}  ${-base_y_size/2 + 0.12}  ${ur5_z_location - 0.03} )" />
   <xacro:arg name="kinect_rpy" default="$(optenv MM_KINECT_RPY 0 0.0 0.0)" />
   <xacro:bare_base/>
   <xacro:ur5_robot prefix="" joint_limited="false"/>
-  <xacro:robotiq_arg2f_140 prefix=""/>
+  <!-- <xacro:robotiq_arg2f_140 prefix=""/> -->
   <joint name="ur_fixed_joint" type="fixed">
     <parent link="bare_base_link" />
@@ -21,9 +21,9 @@
     <origin xyz="${ur5_x_location} 0.0 ${ur5_z_location}" rpy="0.0 0.0 ${M_PI/2}  " />
   </joint>
-  <joint name="ur_gripper_fixed_joint" type="fixed">
+<!--   <joint name="ur_gripper_fixed_joint" type="fixed">
     <parent link="wrist_3_link" />
     <child link = "robotiq_arg2f_base_link" />
     <origin xyz="0.0 ${gripper_z_location_ee} 0.0" rpy="${-M_PI/2} 0.0 0.0  " />
-  </joint>
+  </joint> -->
   <xacro:if value="$(arg kinect_enabled)">
     <joint name="kinect_frame_joint" type="fixed">

Commit message: changed camera_link to kinect1_link

File: mm_description/urdf/mm.urdf.xacro (robot description, xacro)
@@ -30,5 +30,6 @@
       <origin xyz="$(arg kinect_xyz)" rpy="$(arg kinect_rpy)" />
       <parent link="bare_base_link"/>
-      <child link="camera_link"/>
+      <!-- <child link="camera_link"/> -->
+      <child link="kinect1_link"/>
     </joint>
     <xacro:kinect_camera prefix="camera" robot_namespace="$(arg robot_namespace)"/>
