Commit message: post msec push

File: mm_description/urdf/components/bare_base.urdf.xacro (robot description, xacro)
@@ -36,7 +36,7 @@
           <child link="inertial_link" />
         </joint>
-      <link name="world"/>
+      <link name="world2"/>
       <joint name="world_joint" type="floating">
-        <parent link="world"/>
+        <parent link="world2"/>
         <child link="bare_base_link"/>
         <axis xyz="0 0 1" rpy="0 0 0" />
